Commit message: changed urdf to real size, add mass, create first simulation

File: modeling/URDF/motorcycle_witout_loop.urdf.xacro (robot description, xacro)
@@ -1,10 +1,10 @@
 <?xml version="1.0"?>
 <robot xmlns:xacro="http://www.ros.org/wiki/xacro" name="motorcycle">
-    <link name="world"></link>
+    <!-- <link name="world"></link>
     <joint name="base_joint" type="fixed">
         <origin xyz="0.0 0.0 0.0" rpy="0.0 0.0 0.0"/>
         <parent link="world"/>
         <child link="base_link"/>
-    </joint>
+    </joint> -->
     <link name="base_link">
         <inertial>
@@ -122,4 +122,5 @@
         </collision>
     </link>
+<!--
     <link name="right_core_holder_link">
         <inertial>
@@ -213,5 +214,5 @@
             </geometry>
         </collision>
-    </link>
+    </link> -->
     <joint name="front_wheel_joint" type="continuous">
         <origin xyz="0.0 0.0 0.0" rpy="0.0 0.0 0.0"/>
